File: KiCAD/Board/BoardSMD.kicad_sch (KiCad schematic)
At the start: 117 parts, among them J1 MOTOR_5PIN_CONNECTOR, J3 BATTERY_2PIN_CONNECTOR, Q1 AO3400A, Q2 AO3400A, Q3 AO3400A, Q4 AO3400A, Q5 SFH309, Q6 SFH309, U1 4040, U2 7421, U3 74LS393, U4 74HC164, U5 NE555P, U6 ULN2003, U7 ULN2003, U8 LM7805_TO220, U9 NE555P

Commit message: Updated On May 29th 2025
KiCAD Board Almost Done. Will require minor touch ups tomm.
Parts:
- removed C1, C2: C0.1uf, Capacitor_THT:C_Disc_D5.0mm_W2.5mm_P2.50mm, symbol Device:C
- removed C17: C10uf, Capacitor_THT:C_Radial_D6.3mm_H5.0mm_P2.50mm, symbol Device:C
- removed JP1, JP10, JP11, JP12, JP13, JP14, JP15, JP16, JP17, JP18, JP19, JP2, JP20, JP21, JP23, JP3, JP4, JP5, JP6, JP7, JP8, JP9: JMP, Library:Jumper, symbol Jumper:Jumper_2_Open
- removed R2: R4.7K, Resistor_THT:R_Axial_DIN0207_L6.3mm_D2.5mm_P10.16mm_Horizontal, symbol Device:R
- removed SMD_2_DIP1, SMD_2_DIP2, SMD_2_DIP3, SMD_2_DIP4: ~, Library:SMD_2_DIP, symbol New_Library:SMD_2_DIP
- removed U5, U9: NE555P, Package_DIP:DIP-8_W7.62mm, symbol Timer:NE555P
- added J2: DELAY_2PIN_CONNECTOR, Connector_PinSocket_2.54mm:PinSocket_1x02_P2.54mm_Vertical, symbol Connector:Conn_01x02_Socket
- added J4: STATUS_2PIN_CONNECTOR, Connector_PinSocket_2.54mm:PinSocket_1x02_P2.54mm_Vertical, symbol Connector:Conn_01x02_Socket
- added J5: MANUAL_CLK_2PIN_CONNECTOR, Connector_PinSocket_2.54mm:PinSocket_1x02_P2.54mm_Vertical, symbol Connector:Conn_01x02_Socket
- added U5: NE556, Package_DIP:DIP-14_W7.62mm_Socket, symbol Timer:NE556
- C10, C13, C15, C16, C19, C23, C3, C6, C8: footprint Capacitor_THT:C_Radial_D6.3mm_H5.0mm_P2.50mm -> Capacitor_SMD:C_1210_3225Metric_Pad1.33x2.70mm_HandSolder
- C11, C12, C14, C18, C20, C21, C4, C5, C7, C9: footprint Capacitor_THT:C_Disc_D5.0mm_W2.5mm_P2.50mm -> Capacitor_SMD:C_1210_3225Metric_Pad1.33x2.70mm_HandSolder
- D10, D11, D12, D3, D4, D5, D6, D7, D8, D9: footprint Diode_THT:D_DO-35_SOD27_P12.70mm_Horizontal -> Diode_SMD:D_1210_3225Metric
- D14, D15, D16, D17, D2: footprint LED_THT:LED_D3.0mm -> LED_SMD:LED_1210_3225Metric
- J1: footprint Connector_PinSocket_2.54mm:PinSocket_1x05_P2.54mm_Vertical -> Connector_PinSocket_1.27mm:PinSocket_1x05_P1.27mm_Vertical
- R1, R10, R11, R12, R13, R14, R15, R16, R17, R18, R19, R20, R21, R22, R23, R24, R25, R26, R27, R28, R29, R3, R30, R31, R32, R4, R5, R7, R8, R9: footprint Resistor_THT:R_Axial_DIN0207_L6.3mm_D2.5mm_P10.16mm_Horizontal -> Resistor_SMD:R_1210_3225Metric
Connections:
- net 7421_P1 is gone; now on an unnamed net: R10.1
- net 7421_P5 is gone; now on an unnamed net: R9.1
- net ADHOC_LED_5V is gone; now on net +5V: C18.1, C19.1, D2.2 (A), R20.1, R31.1, U4.14 (VCC)
- net AND_VCC is gone; now on net +5V: U2.14 (VCC)
- net MOTOR_CLOCKA is gone; now on an unnamed net: U4.8 (CP)
- net MOTOR_CLOCKB is gone; now on an unnamed net: U3.13 (CP)
- net +5V: now also C12.1, C13.1, J1.1 (Pin_1), R18.1, RV1.3, J2.2 (Pin_2), J5.1 (Pin_1), U5.14 (VCC), U5.14 (VCC), U5.4 (R)
- net DIS_MOTOR: now also U5.13 (DIS)
- net DIS_SYS: now also U5.1 (DIS)
- net GND: now also Q2.3 (D), Q3.3 (D), Q4.3 (D), J4.1 (Pin_1), U5.7 (GND), U5.7 (GND); no longer Q2.2 (S), Q3.2 (S), Q4.2 (S)
- net LOAD: now also R28.1, U3.10 (Q1); no longer U4.2 (DSB)
- net MOTOR1: now also U7.13 (O4); no longer U7.10 (O7)
- net MOTOR2: now also U7.14 (O3); no longer U7.11 (O6)
- net MOTOR3: now also U7.15 (O2); no longer U7.12 (O5)
- net MOTOR4: now also U7.16 (O1); no longer U7.13 (O4)
- net MOTOR_RESET: now also D11.1 (K), D12.1 (K), U5.10 (R)
- net REVERSE_MOTION: now also R29.1, R32.2
- net S0: now also U7.1 (I1)
- net S1: now also U7.2 (I2)
- net S2: now also U7.3 (I3)
- net S3: now also U7.4 (I4)
- net SYSTEM_CLOCK: now also R4.1, U5.5 (Q); no longer U1.10 (CLK)
- net TRIG_MOTOR: now also U5.12 (THR), U5.8 (TR)
- net TRIG_SYS: now also U5.2 (THR), U5.6 (TR)
- net at D14.1 (K), D15.1 (K), D16.1 (K)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: now also J4.2 (Pin_2)
- net MOTOR_CLOCK: now reaches R21.1, R26.1
- net MOTOR_CLOCK: now also U5.9 (Q)
- net at U4.1 (DSA): now also R20.2, U4.9 (~{MR})
- net at Q4.1 (G), R32.1: now also RV3.2; no longer RV3.3
- net at D12.2 (A), Q3.1 (G), Q5.1 (C)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: no longer Q4.3 (D)
- net at R28.2: now also U4.2 (DSB)
- net at R1.2: now also J5.2 (Pin_2)
- net at U6.8 (GND): now also Q3.2 (S); no longer Q3.3 (D)
- net at D10.1 (K), D3.1 (K), D9.1 (K)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: now also D4.1 (K), D5.1 (K), D6.1 (K), D7.1 (K), D8.1 (K)
- net at C22.1: now also RV3.1, J2.1 (Pin_1); no longer RV3.2
- net COMMON_CV: now reaches C14.2
- net COMMON_CV: now also U5.11 (CV), U5.3 (CV)
- net at R4.2: now also U1.10 (CLK)
- net at U7.8 (GND): now also Q2.2 (S); no longer Q2.3 (D)
- net 7421_P2: no longer names the net of R7.1, U2.2
- net 7421_P4: no longer names the net of R8.1, U2.4
Other:
- note removed: "1 = GATE 2 = SOURCE 3 = DRAIN"
- moved on the sheet: Q1, Q2, Q3, Q6, U2A, U3B, U3C, U7
