File: KiCAD/Board/Board.kicad_sch (KiCad schematic)
At the start: 117 parts, among them J1 MOTOR_5PIN_CONNECTOR, J3 BATTERY_2PIN_CONNECTOR, Q1 AO3400A, Q2 AO3400A, Q3 AO3400A, Q4 AO3400A, Q5 SFH309, Q6 SFH309, U1 4040, U2 7421, U3 74LS393, U4 74HC164, U5 NE555P, U6 ULN2003, U7 ULN2003, U8 LM7805_TO220, U9 NE555P

Commit message: Updated on May 30th 2025
Greatly reduced component count and simplified the design and logic of the circuit.
help definitely help with soldering
Parts:
- removed C12, C14: C0.1uf, Capacitor_THT:C_Disc_D5.0mm_W2.5mm_P2.50mm, symbol Device:C
- removed C13, C15, C16, C17: C10uf, Capacitor_THT:C_Radial_D6.3mm_H5.0mm_P2.50mm, symbol Device:C
- removed JP1, JP16, JP17, JP2, JP21, JP3, JP4, JP5: JMP, Library:Jumper, symbol Jumper:Jumper_2_Open
- removed R26: R4.7K, Resistor_THT:R_Axial_DIN0207_L6.3mm_D2.5mm_P10.16mm_Horizontal, symbol Device:R
- removed R30: R10K, Resistor_THT:R_Axial_DIN0207_L6.3mm_D2.5mm_P10.16mm_Horizontal, symbol Device:R
- removed RV1, RV2: POT100K, Potentiometer_THT:Potentiometer_ACP_CA9-H3,8_Horizontal, symbol Device:R_Potentiometer_Trim
- removed U5, U9: NE555P, Package_DIP:DIP-8_W7.62mm, symbol Timer:NE555P
- added C24, C25: C22pF, symbol Device:C
- added C26: C0.1uf, Capacitor_THT:C_Disc_D5.0mm_W2.5mm_P2.50mm, symbol Device:C
- added C27: C10uf, Capacitor_THT:C_Radial_D6.3mm_H5.0mm_P2.50mm, symbol Device:C
- added D18, D19, D20, D21: D4148, Diode_THT:D_DO-35_SOD27_P12.70mm_Horizontal, symbol Device:D
- added R33: R4.7K, Resistor_THT:R_Axial_DIN0207_L6.3mm_D2.5mm_P10.16mm_Horizontal, symbol Device:R
- added R6: R1MEG, symbol Device:R
- added U10: 4015, symbol 4xxx_IEEE:4015
- added U11: CD4060BE, Package_DIP:DIP-16_W7.62mm_Socket, symbol New_Library:CD4060BE
- added U5: 4040, Package_DIP:DIP-16_W7.62mm, symbol 4xxx:4040
- added Y1: Crystal, symbol Device:Crystal
- C2: value C0.1uf -> C10uf; footprint Capacitor_THT:C_Disc_D5.0mm_W2.5mm_P2.50mm -> Capacitor_THT:C_Radial_D6.3mm_H5.0mm_P2.50mm
- R18: value R8.2K -> R4.7K
- R19: value R68K -> R4.7K
Connections:
- net +5V: now also C1.1, C2.1, C26.1, C27.1, U11.16 (VDD), U5.16 (VDD); no longer JP6.2 (B)
- net GND: now also C1.2, C24.2, C25.2, C26.2, C27.2, U11.12 (RESET), U11.8 (VSS), U5.8 (VSS); no longer C1.1, JP7.2 (B)
- net MOTOR_CLOCKB: no longer U3.13 (CP)
- net REVERSE_MOTION: no longer U2.8
- net at R18.1: now also Q1.3 (D), SMD_2_DIP1.3, U2.1, U2.2, U2.4; no longer C2.1
- net at R7.2: no longer U1.14 (Q9)
- net at U1.1 (Q11): now also D18.1 (K); no longer R9.2
- net at U1.15 (Q10): now also D19.1 (K); no longer R8.2
- net at U1.3 (Q4): now also D21.1 (K); no longer R10.2
- net at R21.1: now also U5.4 (Q6)
- net at R21.2: now also U5.11 (Reset)
- net at R3.1, U2.6: now also R19.1
- net at D10.1 (K), D3.1 (K), D9.1 (K)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: now also D7.1 (K), D8.1 (K)
- net at R4.1: now also U2.5, D18.2 (A), D19.2 (A), D20.2 (A), D21.2 (A)
- net at D4.1 (K), D5.1 (K), D6.1 (K): no longer D7.1 (K), D8.1 (K)
- net VCC: now reaches R4.2
- net VCC: now also R18.2
- net 7421_P1: no longer names the net of R10.1
- net 7421_P2: no longer names the net of R7.1
- net 7421_P2: no longer U2.2
- net 7421_P4: no longer names the net of R8.1
- net 7421_P4: no longer U2.4
- net 7421_P5: no longer names the net of R9.1
- removed net DIS_SYS: R18.2, R19.1
- net SYSTEM_CLOCK: no longer names the net of U1.10 (CLK)
- net SYSTEM_CLOCK: now also R33.1
- net TRIG_SYS: no longer names the net of R19.2
- net TRIG_SYS: now also U5.10 (CLK)
- new net: R3.2, U1.11 (Reset)
- new net: D20.1 (K), U1.14 (Q9)
- new net: R33.2, U11.3 (Q14)
- new net: C25.1, R6.2, U11.9 ((PHI)O), Y1.1
- new net: C24.1, R6.1, U11.10 ((PHI)O), Y1.2
- new net: R1.1, U3.1 (CP)
- new net MOTOR_CLOCK: U11.14 (Q8)
Other:
- note added: "Taking Hour-Countdown Clock Pulse from BIT 5 which will be 32 counts made up from 0.5 seconds pulses x 3600 which is half an hour so 32 counts will add up to 16 hours.The Clock pulse at BIT 5 will remain high for another 16 hours until BIT 6 is high at value 64. At that point the counter will reset"

Commit message: May 31st 2025 Updated
Major Design Changed. using LM393 instead of 74HC21 to get half an hour clock signal into hour counter.
connections are more streamlined and easy to solder. Less components as well. went down from 5 mosfets to now just 2 and chips are 6 in total
Parts:
- removed C18, C20, C21: C0.1uf, Capacitor_THT:C_Disc_D5.0mm_W2.5mm_P2.50mm, symbol Device:C
- removed C19, C23: C10uf, Capacitor_THT:C_Radial_D6.3mm_H5.0mm_P2.50mm, symbol Device:C
- removed C22: C100uf, Capacitor_THT:CP_Radial_D10.0mm_P5.00mm, symbol Device:C_Polarized
- removed D11, D12: D4148, Diode_THT:D_DO-35_SOD27_P12.70mm_Horizontal, symbol Device:D
- removed D14, D15, D16, D17: LED, LED_THT:LED_D3.0mm, symbol Device:LED
- removed JP13, JP14, JP15, JP18, JP19, JP23: JMP, Library:Jumper, symbol Jumper:Jumper_2_Open
- removed Q2, Q3, Q4: AO3400A, Package_TO_SOT_SMD:SOT-23, symbol Transistor_FET:AO3400A
- removed Q6: SFH309, LED_THT:LED_D3.0mm_Clear, symbol Sensor_Optical:SFH309
- removed R2, R20, R22, R23, R24, R25, R29, R31, R32: R4.7K, Resistor_THT:R_Axial_DIN0207_L6.3mm_D2.5mm_P10.16mm_Horizontal, symbol Device:R
- removed RV3: POT100K, Potentiometer_THT:Potentiometer_ACP_CA9-H3,8_Horizontal, symbol Device:R_Potentiometer_Trim
- removed SMD_2_DIP1, SMD_2_DIP2, SMD_2_DIP3, SMD_2_DIP4: ~, Library:SMD_2_DIP, symbol New_Library:SMD_2_DIP
- removed U10: 4015, symbol 4xxx_IEEE:4015
- removed U2: 7421, Package_DIP:DIP-14_W7.62mm_Socket, symbol 74xx_IEEE:7421
- removed U3: 74LS393, Package_DIP:DIP-14_W7.62mm_Socket, symbol 74xx:74LS393
- removed U4: 74HC164, Package_DIP:DIP-14_W7.62mm_Socket, symbol 74xx:74HC164
- removed U6, U7: ULN2003, Package_DIP:DIP-16_W7.62mm_Socket, symbol Transistor_Array:ULN2003
- added C12, C14: C10uf, Capacitor_THT:C_Radial_D6.3mm_H5.0mm_P2.50mm, symbol Device:C
- added C13: C0.1uf, Capacitor_THT:C_Disc_D5.0mm_W2.5mm_P2.50mm, symbol Device:C
- added C15: C100uF, Capacitor_THT:CP_Radial_D10.0mm_P5.00mm, symbol Device:C_Polarized
- added D14, D15, D17, D27, D28, D29, D30, D31, D32, D33: D4148, Diode_THT:D_DO-35_SOD27_P12.70mm_Horizontal, symbol Device:D
- added D22, D23, D24, D25, D26: LED, LED_THT:LED_D3.0mm, symbol Device:LED
- added JP1, JP2, JP3, JP4, JP5: JMP, Library:Jumper, symbol Jumper:Jumper_2_Open
- added Q7: AO3400A, Package_TO_SOT_SMD:SOT-23, symbol Transistor_FET:AO3400A
- added Q8: SFH309, LED_THT:LED_D3.0mm_Clear, symbol Sensor_Optical:SFH309
- added R26, R30, R34, R35: R4.7K, Resistor_THT:R_Axial_DIN0207_L6.3mm_D2.5mm_P10.16mm_Horizontal, symbol Device:R
- added RV1: POT100K, Potentiometer_THT:Potentiometer_ACP_CA9-H3,8_Horizontal, symbol Device:R_Potentiometer_Trim
- added U10: ULN2003A, Package_DIP:DIP-16_W7.62mm_Socket, symbol Transistor_Array:ULN2003A
- added U2: 4015, Package_DIP:DIP-16_W7.62mm_Socket, symbol 4xxx_IEEE:4015
- added U3, U9: LM393, Package_DIP:DIP-8_W7.62mm_Socket, symbol Comparator:LM393
- C24, C25: footprint (none) -> Capacitor_THT:C_Disc_D5.0mm_W2.5mm_P2.50mm
- R11, R27: value R10K -> R4.7K
- R13: value R10K -> R47K
- R6: footprint (none) -> Resistor_THT:R_Axial_DIN0207_L6.3mm_D2.5mm_P10.16mm_Horizontal
- U1, U5: footprint Package_DIP:DIP-16_W7.62mm -> Package_DIP:DIP-16_W7.62mm_Socket
- Y1: footprint (none) -> Crystal:Crystal_DS26_D2.0mm_L6.0mm_Vertical
Connections:
- net MOTOR_CLOCK is gone; now on an unnamed net: U11.14 (Q8)
- net S1 is gone; now on net MOTOR_CLOCK_B: JP12.2 (B)
- net S2 is gone; now on net MOTOR_CLOCK_A: JP11.2 (B)
- net S3 is gone; now on an unnamed net: JP10.2 (B)
- net +5V: now also D2.2 (A), JP6.2 (B), R14.2, R17.1, R19.1, R28.1, R9.2, C12.1, C13.1, C14.1, JP1.1 (A), R26.1, U2.16 (Vdd), U2.16 (Vdd), U3.8 (V+), U9.8 (V+); no longer C26.1, C27.1, C7.1, C8.1, U1.16 (VDD), U11.16 (VDD)
- net GND: now also C11.2, R13.1, R27.1, R7.1, C12.2, C13.2, C14.2, C15.2, D22.1 (K), D23.1 (K), D24.1 (K), D25.1 (K), D26.1 (K), Q7.2 (S), Q8.2 (E), R30.1, RV1.2, U10.8 (GND), U2.8 (Vss), U2.8 (Vss), U3.4 (V-), U9.4 (V-); no longer R11.1, R13.2, R27.2
- net MOTOR1: now also U10.16 (O1)
- net MOTOR2: now also U10.15 (O2)
- net MOTOR3: now also U10.14 (O3)
- net MOTOR4: now also U10.13 (O4)
- net REF2.5: now reaches R7.2
- net REF2.5: now also R4.2, U9.3 (+), U9.6 (-)
- net at R3.2: now also D22.2 (A); no longer U1.11 (Reset)
- net Q8: now reaches D10.2 (A), U1.12 (Q8)
- net Q7: now reaches D9.2 (A), U1.13 (Q7)
- net Q0: now reaches D3.2 (A), R5.1, U1.9 (Q0)
- net F1: now reaches JP7.1 (A)
- net F1: now also D14.1 (K), D30.1 (K)
- net F_RESET: now reaches R17.2
- net F_RESET: now also U2.6 (MR), U3.1
- net at R16.1: now also R15.1
- net MOTOR_CLOCK_B: now reaches R16.2
- net MOTOR_CLOCK_A: now reaches R15.2
- net at Q5.1 (C): now also R27.2, Q7.3 (D), R26.2, U3.2 (-)
- net at R9.1: now also JP2.1 (A), JP5.1 (A), U9.1, U9.7
- net at Q1.3 (D): now also R14.1, U2.15 (D), U2.7 (D); no longer R18.1
- net at R28.2: now also R30.2, U3.5 (+); no longer JP9.2 (B)
- net at R1.2: now also Q1.1 (G), R13.2; no longer JP6.1 (A)
- net at R3.1: now also U5.9 (Q0); no longer R19.1
- net at R10.1: now also D23.2 (A)
- net at R10.2: now also U5.7 (Q1)
- net at R12.1: now also D25.2 (A); no longer Q1.1 (G)
- net at JP12.1 (A): now also U2.1 (CP)
- net F2: now reaches JP8.2 (B)
- net F2: now also D29.1 (K), U10.2 (I2)
- net at R1.1: now also D15.1 (K)
- net at JP7.2 (B): now also U10.1 (I1)
- net at D4.1 (K), D5.1 (K), D6.1 (K): now also D7.1 (K), D8.1 (K), JP4.2 (B), U9.2 (-)
- net at U5.10 (CLK): now also JP5.2 (B); no longer R19.2
- net at JP11.1 (A): now also U2.9 (CP)
- net at JP10.1 (A): now also D32.1 (K)
- net at R8.1: now also D18.2 (A), D21.2 (A), JP3.1 (A), U9.5 (+)
- net at R8.2: now also C26.1, C27.1, C7.1, C8.1, JP6.1 (A), R4.1, U1.16 (VDD), U11.16 (VDD)
- net "R" CLOCK: now reaches U5.2 (Q5)
- net "R" CLOCK: now also R34.1, R35.1
- net at U5.3 (Q4): now also R18.2
- net at U5.5 (Q3): now also R12.2
- net at U5.6 (Q2): now also R11.2
- net ADHOC_LED_5V: no longer names the net of JP8.1 (A)
- net ADHOC_LED_5V: now also D33.1 (K); no longer D2.2 (A)
- net LOAD: no longer names the net of JP9.1 (A)
- net LOAD: now also D17.1 (K)
- removed net VCC: R18.2, R4.2
- new net: JP2.2 (B), U1.11 (Reset)
- new net: D14.2 (A), U2.5 (Q1)
- new net: D31.2 (A), D32.2 (A), U2.12 (Q2)
- new net: D28.2 (A), U2.13 (Q1)
- new net: Q8.1 (C), R35.2, U3.6 (-)
- new net: R34.2, U3.3 (+)
- new net: D15.2 (A), D33.2 (A), U2.4 (Q2)
- new net: D27.2 (A), U2.10 (Q4)
- new net: D17.2 (A), U2.3 (Q3)
- new net: D24.2 (A), R11.1
- new net: D10.1 (K), D3.1 (K), D9.1 (K), JP4.1 (A)
- new net: D29.2 (A), U2.11 (Q3)
- new net: D30.2 (A), U2.2 (Q4)
- new net: C15.1, JP1.2 (B), Q7.1 (G), RV1.3
- new net: D19.2 (A), D20.2 (A), JP3.2 (B)
- new net: D26.2 (A), R18.1
- new net F3: D31.1 (K), JP9.2 (B), U10.3 (I3)
- new net F4: D27.1 (K), D28.1 (K), U10.4 (I4)
- new net R_RESET: R19.2, U2.14 (MR), U3.7
Other:
- note removed: "1 = GATE 2 = SOURCE 3 = DRAIN"

Commit message: June 1st Updated
Greatly simplified design using ULN2003 completely and all of its pins. down to only 6 chips and 1 mosfet !!! . This will be  the last design modification. its perfect at this point
Parts:
- removed C13: C0.1uf, Capacitor_THT:C_Disc_D5.0mm_W2.5mm_P2.50mm, symbol Device:C
- removed C14: C10uf, Capacitor_THT:C_Radial_D6.3mm_H5.0mm_P2.50mm, symbol Device:C
- removed JP10, JP7, JP8, JP9: JMP, Library:Jumper, symbol Jumper:Jumper_2_Open
- removed Q1: AO3400A, Package_TO_SOT_SMD:SOT-23, symbol Transistor_FET:AO3400A
- removed Q8: SFH309, LED_THT:LED_D3.0mm_Clear, symbol Sensor_Optical:SFH309
- removed R17, R19, R26, R27, R28, R30, R34, R35: R4.7K, Resistor_THT:R_Axial_DIN0207_L6.3mm_D2.5mm_P10.16mm_Horizontal, symbol Device:R
- removed U3: LM393, Package_DIP:DIP-8_W7.62mm_Socket, symbol Comparator:LM393
- added D11, D12: D4148, Diode_THT:D_DO-35_SOD27_P12.70mm_Horizontal, symbol Device:D
- added Q1: SFH309, LED_THT:LED_D3.0mm_Clear, symbol Sensor_Optical:SFH309
- added R2, R22, R23: R4.7K, Resistor_THT:R_Axial_DIN0207_L6.3mm_D2.5mm_P10.16mm_Horizontal, symbol Device:R
- added R20: R47K, Resistor_THT:R_Axial_DIN0207_L6.3mm_D2.5mm_P10.16mm_Horizontal, symbol Device:R
- R13: value R47K -> R4.7K
Connections:
- net "R" CLOCK: now also R14.1, R2.2
- net +5V: now also R1.2, R13.2, R22.2, R23.2; no longer R14.2
- net F1: now also U10.1 (I1)
- net F2: now also D33.1 (K)
- net F3: now also D17.1 (K)
- net F_RESET: now also U10.10 (O7), D12.2 (A), R22.1; no longer U2.6 (MR)
- net GND: now also Q1.2 (E), R20.2; no longer R13.1
- net R_RESET: now also R13.1, U10.11 (O6)
- net LOAD: now reaches U2.15 (D), U2.7 (D)
- net LOAD: now also R1.1, U10.12 (O5); no longer R14.1
- net at Q5.1 (C): now also U10.6 (I6), R2.1; no longer Q7.3 (D)
- net at D15.1 (K): now also D32.1 (K), U10.5 (I5); no longer R1.1
- net at U10.7 (I7): now also Q7.3 (D), Q1.1 (C), R23.1
- new net: D11.2 (A), R14.2
- new net: D11.1 (K), D12.1 (K), R20.1, U2.6 (MR)
Other:
- moved on the sheet: C15, Q7, RV1, U10, U2A, U2B

Commit message: June 1st Project COMPLETED
Project Completed and Ready for Soldering
Parts:
- removed JP12: JMP, Library:Jumper, symbol Jumper:Jumper_2_Open
- added J2: MOTOR_5PIN_CONNECTOR_2, Connector_PinSocket_2.54mm:PinSocket_1x05_P2.54mm_Vertical, symbol Connector:Conn_01x05_Pin
- added JP10, JP13, JP14, JP15, JP16, JP17, JP19, JP21, JP7, JP8, JP9: JMP, Library:Jumper, symbol Jumper:Jumper_2_Open
- added R17: R4.7K, Resistor_THT:R_Axial_DIN0207_L6.3mm_D2.5mm_P10.16mm_Horizontal, symbol Device:R
Connections:
- net +5V: now also C26.1, C27.1, C7.1, C8.1, J1.1 (Pin_1), JP20.1 (A), JP6.1 (A), R4.1, R8.2, U1.16 (VDD), U11.16 (VDD), J2.5 (Pin_5), JP19.2 (B); no longer C1.1, C10.1, C2.1, C9.1, D1.2 (A), D13.2 (A), D2.2 (A), JP20.2 (B), JP6.2 (B), R9.2, U5.16 (VDD), U9.8 (V+)
- net F1: now also JP15.2 (B); no longer U10.1 (I1)
- net F2: now also JP17.1 (A); no longer D33.1 (K)
- net F3: now also JP16.1 (A); no longer D17.1 (K)
- net F_RESET: now also JP14.1 (A); no longer D12.2 (A)
- net GND: now also JP21.2 (B); no longer U9.4 (V-)
- net LOAD: now also JP9.2 (B); no longer R1.1, U10.12 (O5)
- net MOTOR1: now also J2.4 (Pin_4)
- net MOTOR2: now also J2.3 (Pin_3)
- net MOTOR3: now also J2.2 (Pin_2)
- net MOTOR4: now also J2.1 (Pin_1)
- net MOTOR_CLOCK_B: now also U2.1 (CP)
- net R_RESET: now also JP10.1 (A); no longer R13.1, U10.11 (O6)
- net at D11.2 (A): now also JP8.1 (A); no longer R14.2
- net at Q5.1 (C), U10.6 (I6): now also JP7.2 (B); no longer R2.1
- net at JP5.2 (B), U5.10 (CLK): now also R17.1
- net at D32.1 (K), U10.5 (I5): now also JP13.2 (B); no longer D15.1 (K)
- net "R" CLOCK: no longer names the net of R14.1, U5.2 (Q5)
- net "R" CLOCK: now also R2.1; no longer R2.2
- new net: JP9.1 (A), R1.1, U10.12 (O5)
- new net: D33.1 (K), JP17.2 (B)
- new net: D12.2 (A), JP14.2 (B)
- new net: D2.2 (A), JP19.1 (A), R9.2
- new net: JP21.1 (A), U9.4 (V-)
- new net: JP15.1 (A), U10.1 (I1)
- new net: JP10.2 (B), R13.1, U10.11 (O6)
- new net: JP6.2 (B), R17.2
- new net: D15.1 (K), JP13.1 (A)
- new net: D17.1 (K), JP16.2 (B)
- new net "R" CLOCK A: JP7.1 (A), R14.2
- new net "R" CLOCK B: JP8.2 (B), R2.2
- new net CLK_VCC: C1.1, C10.1, C2.1, C9.1, D1.2 (A), D13.2 (A), JP20.2 (B), U5.16 (VDD), U9.8 (V+)
Other:
- moved on the sheet: C15, Q7, RV1, U10, U2A, U2B
